File: HeatTable-Base-v0.9/HeatTable-Base-v0.9.kicad_sch (KiCad schematic)
At the start: 81 parts, among them J1 DC-005-5A-2.5, J2 2x10xP1.27mm, J3 DEBUG, J4 1x03x2.54mm, J5 1.25mm SMD, J6 2x10x1.27mm_SMD, J7 2x10x1.27mm_SMD, J8 2x10x1.27mm_SMD, J9 2x10x1.27mm_SMD, Q1 WSP4409A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

Commit message: modified the USB C footprint for better hand soldering
Parts:
- USB1: footprint User:USB_C_Receptacle_HRO_TYPE-C-31-M-17 -> User:USB_C_Receptacle_HRO_TYPE-C-31-M-17_Handsoldering
Changed lines of the file:
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@@
     (property "Reference" "USB1" (id 0) (at 83.82 21.59 0))
     (property "Value" "TYPE-C-31-M-17" (id 1) (at 83.82 24.13 0))
-    (property "Footprint" "User:USB_C_Receptacle_HRO_TYPE-C-31-M-17" (id 2) (at 87.63 44.45 0)
+    (property "Footprint" "User:USB_C_Receptacle_HRO_TYPE-C-31-M-17_Handsoldering" (id 2) (at 87.63 44.45 0)
       (effects (font (size 1.27 1.27)) hide)
     )
@@
     )
     (path "/7f2e95a6-c747-4b57-b6d7-1d71ac4dfaa0"
-      (reference "USB1") (unit 1) (value "TYPE-C-31-M-17") (footprint "User:USB_C_Receptacle_HRO_TYPE-C-31-M-17")
-    )
-  )
+      (reference "USB1") (unit 1) (value "TYPE-C-31-M-17") (footprint "User:USB_C_Receptacle_HRO_TYPE-C-31-M-17_Handsoldering")
+    )
+  )
